File: range/sensor/sensor.sch (KiCad schematic (older format))
At the start: 7 parts, among them P1 CONN_2

Commit message: had a go at creating a piezo board and gerbers
Changed lines of the file:
@@
 $EndComp
 $Comp
-L GND #PWR?
+L GND #PWR01
 U 1 1 54CFE05E
 P 5500 4000
-F 0 "#PWR?" H 5500 4000 30  0001 C CNN
+F 0 "#PWR01" H 5500 4000 30  0001 C CNN
 F 1 "GND" H 5500 3930 30  0001 C CNN
 F 2 "" H 5500 4000 60  0000 C CNN
@@
 $EndComp
 Wire Wire Line
-	3800 3100 4100 3100
+	3800 3100 5800 3100
 Wire Wire Line
-	4100 3100 4450 3100
+	5500 3600 5500 4000
 Wire Wire Line
-	4450 3100 4800 3100
-Wire Wire Line
-	4800 3100 5150 3100
-Wire Wire Line
-	5150 3100 5500 3100
-Wire Wire Line
-	5500 3100 5800 3100
-Wire Wire Line
-	5500 3600 5500 3900
-Wire Wire Line
-	5500 3900 5500 4000
-Wire Wire Line
-	3100 3900 4100 3900
-Wire Wire Line
-	4100 3900 4450 3900
-Wire Wire Line
-	4450 3900 4800 3900
-Wire Wire Line
-	4800 3900 5150 3900
-Wire Wire Line
-	5150 3900 5500 3900
-Wire Wire Line
-	5500 3900 5800 3900
+	3100 3900 5800 3900
 Wire Wire Line
 	4100 3350 4100 3100
